File: Hardware/LilyPad-Dev-v34.brd (EAGLE design)
At the start: 104.1 x 72.4 mm, 156 parts, among them M1 MOTORSMD, U1 ATMEGA328, U2 MCP9700, U3 TEMT6000, U4 MCP73831, Y1 8MHz

Commit message: Adding current board files
Parts:
- removed TP2: (no value), SparkFun:PAD.03X.05
- C1, C10, C3, C4, C9: device SparkFun:0603-CAP -> SparkFun:0402-CAP
- D1, D4: device SparkFun-LED:LED-0603-QC -> SparkFun:LED-0603
- R1, R12, R2, R3, R4, R5, R6: device SparkFun:0603-RES -> SparkFun:0402-RES
- R13: value 1k -> 10k; device SparkFun:0603-RES -> SparkFun:0402-RES
- R7: device SparkFun:0603-RES -> SparkFun:C0402
- moved D4 0.76 mm to (44.9, 40.1)
- moved R4 0.51 mm to (12.7, 32.3)
- moved R12 0.51 mm to (43.7, 40.0)
- moved R5 0.46 mm to (16.6, 34.6)
- moved R3 0.40 mm to (8.80, 34.6)
- moved C3 0.36 mm to (45.1, 49.0)
- moved R6 0.36 mm to (18.5, 55.7)
- moved C9 0.25 mm to (37.7, 40.0)
- moved R13 0.25 mm to (42.5, 40.0)
- moved U4 0.25 mm to (40.1, 40.0)
- moved Y1 0.13 mm to (45.2, 45.0)
Connections:
- net VBATT: no longer TP2.P$1
Routing:
- net GND: track 463.5 -> 460.9 mm
- net D3: track 52.4 -> 54.0 mm
- net VBATT: track 31.0 -> 29.7 mm, vias 1 -> 0
- net VCC: track 300.1 -> 299.0 mm
- net RST: track 37.4 -> 36.4 mm
- net STAT: track 4.22 -> 3.27 mm
- net PROG: track 1.64 -> 2.32 mm
- net GRN: track 2.58 -> 3.24 mm
- net RED: track 5.53 -> 6.12 mm
- net FTDI_VCC: track 58.9 -> 59.5 mm
Other:
- board text added: "v34"
- board text removed: "v35"
