File: Hardware/LilyPad-Dev-v34.sch (EAGLE design)
At the start: 138 parts, among them M1 MOTORSMD, U1 ATMEGA328, U2 MCP9700, U3 TEMT6000, U4 MCP73831, Y1 8MHz

Commit message: Adding current board files
Parts:
- removed TP2: TEST-POINT3X5, SparkFun:TEST-POINT3X5
- C1, C10, C3, C4, C9: device SparkFun:CAP0603-CAP -> SparkFun:CAP0402-CAP
- D1, D4: device SparkFun-LED:LEDQC -> SparkFun:LED0603
- R1, R12, R2, R3, R4, R5, R6, R7: device SparkFun:RESISTOR0603-RES -> SparkFun:RESISTOR0402-RES
- R13: value 1k -> 10k; device SparkFun:RESISTOR0603-RES -> SparkFun:RESISTOR0402-RES
Connections:
- net VBATT: no longer TP2.1
Other:
- note removed: "-Changed all componets to true 0603 packages"
- note removed: "-added test point for lipo batt input"
- note removed: "Changes to V35 (5/4/2012)"
