File: Hardware/ProtoSnap-LilyPad_Development_Board.sch (EAGLE design)
At the start: 138 parts, among them M1 MOTORSMD, U1 ATMEGA328, U2 MCP9700, U3 TEMT6000, U4 MCP73831, Y1 8MHz

Commit message: finishing up v35 - a few things
-updated LILYPAD-BRD-LAYERS.pac to include fixed polygons.
-updated to ledger in schematic, updated "designed by" text objects.
re-spaced schematic for more even look
-updated to 1:1 (+fake traces) footprint on resonator package
Parts:
- added FRAME2: FRAME-LEDGER, SparkFun-Aesthetics:FRAME-LEDGER
- BUTTON-, BUTTONS, SLIDEOFF, SLIDEON: device LilyPad-Wearables:SEWTAP4 -> LilyPad-Wearables:SEWTAP8
- LIGHT+, LIGHT-, LIGHTS, TEMP+, TEMP-, TEMPS, U$32-, U$33+, VIBE+, VIBE-: device LilyPad-Wearables:SEWTAP4 -> LilyPad-Wearables:SEWTAP6
- Y1: device SparkFun:RESONATORSMD -> Testing:RESONATOR1:1
Other:
- note added: "35"
- note removed: "Designed by:"
- note removed: "LilyPad - MainBoard Simple"
- note removed: "Released under the Creative Commons Attribution Share-Alike 3.0 License"
- note removed: "http://creativecommons.org/licenses/by-sa/3.0"
- moved on the sheet: B1, C1, C10, C2, C3, C4, C5, C9, D1, D2, D3, D4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

Commit message: Added diode from VBATT to VBUS
also updated to flags in schematic.
Parts:
- added D5: B340A, SparkFun-DiscreteSemi:DIODE-SCHOTTKY_
- D1, D4: device SparkFun-LED:LEDQC -> Testing:LEDLED-ALT1
- S4: device SparkFun:SWITCH-MOMENTARY-2SMD -> Testing:SWITCH-MOMENTARY-2SMD-ALT01
Connections:
- removed net N$12: U1.PD4(XCK/T0)
- removed net N$14: U1.PB0(ICP)
- removed net N$5: U1.PC0(ADC0)
- removed net N$8: U1.ADC7
- net FTDI_VCC: now also D5.C
- net VBATT: now also D5.A
Other:
- note removed: "-Changed all componets to true 0603 packages"
- note removed: "-added OSHL to main board"
- note removed: "-added more perferation drills on tabs for easier cutting"
- note removed: "-added test point for lipo batt input"
- note removed: "-changed lots of silk to vector style font"
- note removed: "-fixed miso line"
- note removed: "-modified demension on all outer boards to make for easier snapping"
- note removed: "-moved to SMD vibe motor"
- note removed: "Changes to V33 (12/22/11)"
- note removed: "Changes to V34 (1/9/2012)"
- note removed: "Changes to V35 (5/4/2012)"
- moved on the sheet: C10, C9, D4, R12, R13, TP-DTR, TP-RX, TP-TX, U4

Commit message: Updated momentary buttons to new package
Parts:
- S3: value (none) -> SWITCH-MOMENTARY-2SMD-REDUNDANT; device SparkFun:TAC_SWITCHSMD -> SparkFun-Electromechanical:SWITCH-MOMENTARY-2SMD-REDUNDANT
- S4: device Testing:SWITCH-MOMENTARY-2SMD-ALT01 -> SparkFun-Electromechanical:SWITCH-MOMENTARY-2SMD-REDUNDANT
Connections:
- net A5: now also S3.1; no longer S3.2
- net GND: now also S3.2; no longer S3.4
Changed lines of the file:
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@@
 <layer number="54" name="bGND_GNDA" color="1" fill="9" visible="no" active="no"/>
 <layer number="56" name="wert" color="7" fill="1" visible="no" active="no"/>
+<layer number="57" name="tCAD" color="7" fill="1" visible="no" active="no"/>
 <layer number="91" name="Nets" color="2" fill="1" visible="yes" active="yes"/>
 <layer number="92" name="Busses" color="1" fill="1" visible="yes" active="yes"/>
@@
 <layer number="97" name="Info" color="7" fill="1" visible="yes" active="yes"/>
 <layer number="98" name="Guide" color="6" fill="1" visible="yes" active="yes"/>
+<layer number="99" name="SpiceOrder" color="7" fill="1" visible="yes" active="yes"/>
 <layer number="100" name="Muster" color="7" fill="1" visible="no" active="no"/>
 <layer number="101" name="Patch_Top" color="12" fill="4" visible="yes" active="yes"/>
@@
 <layer number="108" name="tplace-old" color="10" fill="1" visible="yes" active="yes"/>
 <layer number="109" name="ref-old" color="11" fill="1" visible="yes" active="yes"/>
+<layer number="110" name="fp0" color="7" fill="1" visible="yes" active="yes"/>
+<layer number="111" name="LPC17xx" color="7" fill="1" visible="yes" active="yes"/>
+<layer number="112" name="tSilk" color="7" fill="1" visible="yes" active="yes"/>
 <layer number="116" name="Patch_BOT" color="9" fill="4" visible="yes" active="yes"/>
 <layer number="121" name="_tsilk" color="7" fill="1" visible="yes" active="yes"/>
 <layer number="122" name="_bsilk" color="7" fill="1" visible="yes" active="yes"/>
+<layer number="123" name="tTestmark" color="7" fill="1" visible="yes" active="yes"/>
+<layer number="124" name="bTestmark" color="7" fill="1" visible="yes" active="yes"/>
 <layer number="125" name="_tNames" color="7" fill="1" visible="yes" active="yes"/>
+<layer number="126" name="_bNames" color="7" fill="1" visible="yes" active="yes"/>
+<layer number="127" name="_tValues" color="7" fill="1" visible="yes" active="yes"/>
+<layer number="128" name="_bValues" color="7" fill="1" visible="yes" active="yes"/>
+<layer number="131" name="tAdjust" color="7" fill="1" visible="yes" active="yes"/>
+<layer number="132" name="bAdjust" color="7" fill="1" visible="yes" active="yes"/>
 <layer number="144" name="Drill_legend" color="7" fill="1" visible="yes" active="yes"/>
+<layer number="150" name="Notes" color="7" fill="1" visible="yes" active="yes"/>
 <layer number="151" name="HeatSink" color="7" fill="1" visible="yes" active="yes"/>
+<layer number="152" name="_bDocu" color="7" fill="1" visible="yes" active="yes"/>
+<layer number="153" name="FabDoc1" color="7" fill="1" visible="yes" active="yes"/>
+<layer number="154" name="FabDoc2" color="7" fill="1" visible="yes" active="yes"/>
+<layer number="155" name="FabDoc3" color="7" fill="1" visible="yes" active="yes"/>
 <layer number="199" name="Contour" color="7" fill="1" visible="yes" active="yes"/>
 <layer number="200" name="200bmp" color="1" fill="10" visible="no" active="no"/>
@@
 <layer number="223" name="223bmp" color="24" fill="1" visible="no" active="no"/>
 <layer number="224" name="224bmp" color="25" fill="1" visible="no" active="no"/>
+<layer number="248" name="Housing" color="7" fill="1" visible="yes" active="yes"/>
+<layer number="249" name="Edge" color="7" fill="1" visible="yes" active="yes"/>
 <layer number="250" name="Descript" color="3" fill="1" visible="no" active="no"/>
 <layer number="251" name="SMDround" color="12" fill="11" visible="no" active="no"/>
@@
 <part name="P+8" library="SparkFun" deviceset="VCC" device=""/>
 <part name="GND12" library="supply1" deviceset="GND" device=""/>
-<part name="S4" library="Testing" deviceset="SWITCH-MOMENTARY-2" device="SMD-ALT01" value="Reset"/>
+<part name="S4" library="SparkFun-Electromechanical" deviceset="SWITCH-MOMENTARY-2" device="SMD-REDUNDANT" value="Reset"/>
 <part name="PP-MISO" library="SparkFun" deviceset="TEST-POINT" device="3X5" value=""/>
 <part name="PP-SCK" library="SparkFun" deviceset="TEST-POINT" device="3X5" value=""/>
@@
 <part name="SLIDEOFF" library="LilyPad-Wearables" deviceset="SEWTAP" device="8" value="SEWTAP8"/>
 <part name="SLIDEON" library="LilyPad-Wearables" deviceset="SEWTAP" device="8" value="SEWTAP8"/>
-<part name="S3" library="SparkFun" deviceset="TAC_SWITCH" device="SMD"/>
 <part name="BUTTONS" library="LilyPad-Wearables" deviceset="SEWTAP" device="8" value="SEWTAP8"/>
 <part name="BUTTON-" library="LilyPad-Wearables" deviceset="SEWTAP" device="8" value="SEWTAP8"/>
@@
 <part name="FRAME2" library="SparkFun-Aesthetics" deviceset="FRAME-LEDGER" device=""/>
 <part name="D5" library="SparkFun-DiscreteSemi" deviceset="DIODE-SCHOTTKY" device="_" value="B340A"/>
+<part name="S3" library="SparkFun-Electromechanical" deviceset="SWITCH-MOMENTARY-2" device="SMD-REDUNDANT" value=""/>
 </parts>
 <sheets>
@@
 <wire x1="73.66" y1="81.28" x2="43.18" y2="81.28" width="0.2032" layer="94"/>
 <wire x1="45.72" y1="114.3" x2="40.64" y2="109.22" width="0.2032" layer="94" curve="90"/>
-<wire x1="40.64" y1="109.22" x2="40.64" y2="101.6" width="0.2032" layer="94"/>
-<wire x1="40.64" y1="101.6" x2="45.72" y2="96.52" width="0.2032" layer="94" curve="90"/>
-<wire x1="45.72" y1="96.52" x2="71.12" y2="96.52" width="0.2032" layer="94"/>
-<wire x1="71.12" y1="96.52" x2="76.2" y2="101.6" width="0.2032" layer="94" curve="90"/>
-<wire x1="76.2" y1="101.6" x2="76.2" y2="109.22" width="0.2032" layer="94"/>
+<wire x1="40.64" y1="109.22" x2="40.64" y2="104.14" width="0.2032" layer="94"/>
+<wire x1="40.64" y1="104.14" x2="45.72" y2="99.06" width="0.2032" layer="94" curve="90"/>
+<wire x1="45.72" y1="99.06" x2="71.12" y2="99.06" width="0.2032" layer="94"/>
+<wire x1="71.12" y1="99.06" x2="76.2" y2="104.14" width="0.2032" layer="94" curve="90"/>
+<wire x1="76.2" y1="104.14" x2="76.2" y2="109.22" width="0.2032" layer="94"/>
 <wire x1="76.2" y1="109.22" x2="71.12" y2="114.3" width="0.2032" layer="94" curve="90"/>
 <wire x1="71.12" y1="114.3" x2="45.72" y2="114.3" width="0.2032" layer="94"/>
@@
 <instance part="SLIDEOFF" gate="G$1" x="38.1" y="71.12" rot="R180"/>
 <instance part="SLIDEON" gate="G$1" x="76.2" y="73.66"/>
-<instance part="S3" gate="S" x="58.42" y="104.14"/>
-<instance part="BUTTONS" gate="G$1" x="48.26" y="101.6" rot="R180"/>
-<instance part="BUTTON-" gate="G$1" x="68.58" y="101.6"/>
+<instance part="BUTTONS" gate="G$1" x="48.26" y="106.68" rot="R180"/>
+<instance part="BUTTON-" gate="G$1" x="68.58" y="106.68"/>
 <instance part="R" gate="G$1" x="180.34" y="38.1" rot="R270"/>
 <instance part="LED+" gate="G$1" x="180.34" y="55.88" rot="R90"/>
@@
 <instance part="FRAME2" gate="G$2" x="330.2" y="0"/>
 <instance part="D5" gate="G$1" x="208.28" y="129.54" rot="R180"/>
+<instance part="S3" gate="G$1" x="58.42" y="106.68"/>
 </instances>
 <busses>
@@
 </segment>
 <segment>
-<wire x1="66.04" y1="101.6" x2="63.5" y2="101.6" width="0.1524" layer="91"/>
-<pinref part="S3" gate="S" pin="4"/>
+<wire x1="66.04" y1="106.68" x2="63.5" y2="106.68" width="0.1524" layer="91"/>
 <pinref part="BUTTON-" gate="G$1" pin="1"/>
+<pinref part="S3" gate="G$1" pin="2"/>
 </segment>
 <segment>
@@
 </segment>
 <segment>
-<wire x1="50.8" y1="101.6" x2="53.34" y2="101.6" width="0.1524" layer="91"/>
-<pinref part="S3" gate="S" pin="2"/>
+<wire x1="50.8" y1="106.68" x2="53.34" y2="106.68" width="0.1524" layer="91"/>
 <pinref part="BUTTONS" gate="G$1" pin="1"/>
-</segment>
-<segment>
+<pinref part="S3" gate="G$1" pin="1"/>
+</segment>
+<segment>

Commit message: Replaced resonator device to SparkFun-FreqCtrl.lbr
This used to be from SFE-testing-library, and now it's linked to the
"official/proven" SFE library.
Parts:
- Y1: device Testing:RESONATOR1:1 -> SparkFun-FreqCtrl:RESONATOR8MHZ
Changed lines of the file:
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@@
 <part name="GND3" library="SparkFun" deviceset="GND" device=""/>
 <part name="GND4" library="SparkFun" deviceset="GND" device=""/>
-<part name="Y1" library="Testing" deviceset="RESONATOR" device="1:1" value="8MHz"/>
+<part name="Y1" library="SparkFun-FreqCtrl" deviceset="RESONATOR" device="8MHZ" value="8MHz"/>
 <part name="GND9" library="SparkFun" deviceset="GND" device=""/>
 <part name="JP2" library="SparkFun" deviceset="ARDUINO_SERIAL_PROGRAM" device="SMD"/>

Commit message: Schematic cleanup and a few brd part nudges
-Fixed 4 way junction in reset net.
-Moved a few vias, and parts to avoid DRC clearance errors.
Other:
- moved on the sheet: S4
Changed lines of the file:
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@@
 <attribute name="VALUE" x="189.484" y="216.916" size="1.778" layer="96"/>
 </instance>
-<instance part="GND6" gate="1" x="190.5" y="180.34"/>
+<instance part="GND6" gate="1" x="187.96" y="180.34"/>
 <instance part="P+3" gate="1" x="200.66" y="205.74" smashed="yes">
 <attribute name="VALUE" x="199.644" y="209.296" size="1.778" layer="96"/>
@@
 </instance>
 <instance part="GND12" gate="1" x="154.94" y="208.28"/>
-<instance part="S4" gate="G$1" x="190.5" y="190.5" rot="R90"/>
+<instance part="S4" gate="G$1" x="187.96" y="190.5" rot="R90"/>
 <instance part="PP-MISO" gate="G$1" x="162.56" y="175.26" smashed="yes" rot="R180">
 <attribute name="NAME" x="148.082" y="174.498" size="1.778" layer="95"/>
@@
 </segment>
 <segment>
-<wire x1="190.5" y1="185.42" x2="190.5" y2="182.88" width="0.1524" layer="91"/>
+<wire x1="187.96" y1="185.42" x2="187.96" y2="182.88" width="0.1524" layer="91"/>
 <pinref part="GND6" gate="1" pin="GND"/>
 <pinref part="S4" gate="G$1" pin="1"/>
@@
 <segment>
 <wire x1="190.5" y1="200.66" x2="190.5" y2="198.12" width="0.1524" layer="91"/>
-<wire x1="190.5" y1="198.12" x2="190.5" y2="195.58" width="0.1524" layer="91"/>
+<wire x1="190.5" y1="198.12" x2="187.96" y2="198.12" width="0.1524" layer="91"/>
+<wire x1="187.96" y1="198.12" x2="187.96" y2="195.58" width="0.1524" layer="91"/>
 <wire x1="190.5" y1="198.12" x2="203.2" y2="198.12" width="0.1524" layer="91"/>
-<wire x1="185.42" y1="198.12" x2="190.5" y2="198.12" width="0.1524" layer="91"/>
+<wire x1="185.42" y1="198.12" x2="187.96" y2="198.12" width="0.1524" layer="91"/>
 <junction x="190.5" y="198.12"/>
 <label x="193.04" y="198.12" size="1.778" layer="95"/>
@@
 <pinref part="C4" gate="G$1" pin="2"/>
 <pinref part="S4" gate="G$1" pin="2"/>
-</segment>
-<segment>
+<junction x="187.96" y="198.12"/>
+<wire x1="187.96" y1="198.12" x2="190.5" y2="198.12" width="0.1524" layer="91"/>
+</segment>
+<segment>

Commit message: Common Cathode LED, ALS-PT19 light sensor
Also added measures and "route out" text.
Parts:
- removed D2: LED-TRICOLOR, SparkFun:LED-TRICOLOR
- removed R3: 200, SparkFun:RESISTOR0603-RES
- removed R4, R5: 100, SparkFun:RESISTOR0603-RES
- removed U3: TEMT6000, SparkFun:TEMT6000
- added D6: LED-TRICOLOR, SparkFun-LED:LED-TRICOLOR-NO-COMPLCC-6-SMD
- added R17: 300, SparkFun-Resistors:300OHM-1/10W-1%(0603)
- added R19, R21: 100, SparkFun-Resistors:100OHM1/10W1%(0603)
- added U6: LIGHTSENSOR_ALS-PT19, SparkFun-Sensors:LIGHTSENSORALS
- U$48: value MOUSE-BITE-3(NO_PADS) -> MOUSE-BITE-2; device Testing:MOUSE-BITE-3(NO_PADS) -> Testing:MOUSE-BITE-2
- renumbered FRAME2 to FRAME1
Connections:
- removed net BLU: D2.BLU, R4.2
- removed net GRN: D2.GRN, R5.2
- removed net RED: D2.RED, R3.2
- new net BLUE: D6.BC, R17.2
- new net GRN1: D6.GC, R21.2
- new net RED1: D6.RC, R19.2
- net A6: now also U6.E1; no longer U3.E1
- net D10: now also D6.BLU, U$20.P$3; no longer R4.1, U$20.P$2
- net D11: now also D6.GRN, U$20.P$2; no longer R5.1, U$20.P$1
- net D9: now also D6.RED, U$20.P$4; no longer R3.1, U$20.P$3
- net GND: now also R17.1, R19.1, R21.1, U$25.1, U$48.P$1
- net VCC: now also U6.C1; no longer D2.A, U$20.P$4, U$25.1, U3.C1
Other:
- note added: "RGB LED"
- moved on the sheet: D3, M1, R6, R7, S2, S3

Commit message: more schematic cleanup
Parts:
- removed LED, LED1, LED2, LED3, LED4: White, SparkFun-3-2-07:LED1206
- added D10: LED-TRICOLOR, SparkFun-LED:LED-TRICOLOR-NO-COMPLCC-6-SMD
- added D2: White, SparkFun-3-2-07:LED1206
- added D7: Yellow, Testing:LEDLED-ALT1
- added D8: B340A, SparkFun-DiscreteSemi:DIODE-SCHOTTKY_
- added D9: (no value), SparkFun:DIODESOD
- D3: value (none) -> White; device SparkFun:DIODESOD -> SparkFun-3-2-07:LED1206
- D4: value Yellow -> White; device Testing:LEDLED-ALT1 -> SparkFun-3-2-07:LED1206
- D5: value B340A -> White; device SparkFun-DiscreteSemi:DIODE-SCHOTTKY_ -> SparkFun-3-2-07:LED1206
- D6: value LED-TRICOLOR -> White; device SparkFun-LED:LED-TRICOLOR-NO-COMPLCC-6-SMD -> SparkFun-3-2-07:LED1206
- M1: value MOTORSMD -> VIBE MOTOR
Connections:
- net BLUE: now also D10.BC; no longer D6.BC
- net D10: now also D10.BLU; no longer D6.BLU
- net D11: now also D10.GRN; no longer D6.GRN
- net D9: now also D10.RED; no longer D6.RED
- net FTDI_VCC: now also D7.A, D8.C; no longer D4.A, D5.C
- net GND: now also D9.A; no longer D3.A
- net GRN1: now also D10.GC; no longer D6.GC
- net N$10: now also D9.C; no longer D3.C
- net N$18: now also D2.C; no longer LED.C
- net N$19: now also D2.A; no longer LED.A
- net N$21: now also D3.C; no longer LED1.C
- net N$22: now also D3.A; no longer LED1.A
- net N$24: now also D4.C; no longer LED2.C
- net N$25: now also D4.A; no longer LED2.A
- net N$27: now also D5.C; no longer LED3.C
- net N$28: now also D5.A; no longer LED3.A
- net N$30: now also D6.C; no longer LED4.C
- net N$31: now also D6.A; no longer LED4.A
- net N$33: now also D7.C; no longer D4.C
- net RED1: now also D10.RC; no longer D6.RC
- net VBATT: now also D8.A; no longer D5.A
Other:
- note added: "Programming Testpoints"
- note removed: "RGB LED"
- moved on the sheet: D4, M1, PP-GND, PP-MISO, PP-RST, PP-SCK, R6, TP1

Commit message: removed sheet 2
had notes about old revisions, this is now unnecessary
Other:
- note removed: "-Changed Buzzer from D12/D7 to GND/D7, for easier buzzing."
- note removed: "-Changes to v32 (9/26/2011)"
- note removed: "-Fixed Silk error on RGB LED"
- note removed: "-Swapped silk for LEDs (A3 and A4 were backwards)"
Changed lines of the file:
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@@
-</nets>
-</sheet>
-<sheet>
-<plain>
-<text x="2.54" y="27.94" size="1.778" layer="94">-Changes to v32 (9/26/2011)</text>
-<text x="7.62" y="25.4" size="1.778" layer="94">-Fixed Silk error on RGB LED</text>
-<text x="7.62" y="22.86" size="1.778" layer="94">-Swapped silk for LEDs (A3 and A4 were backwards)</text>
-<text x="7.62" y="20.32" size="1.778" layer="94">-Changed Buzzer from D12/D7 to GND/D7, for easier buzzing.</text>
-</plain>
-<instances>
-</instances>
-<busses>
-</busses>
-<nets>
 </nets>
 </sheet>
